Commit message: rexrov with multibeam sonar displayed in rviz

File: rexrov2_description/urdf/rexrov2_sensors.xacro (robot description, xacro)
@@ -70,3 +70,18 @@
     <origin xyz="0 0 0" rpy="0 0 0"/>
   </xacro:default_chemical_concentration_sensor_macro>
+  <!-- Forward-looking sonar sensor -->
+  <xacro:forward_looking_sonar
+    namespace="${namespace}"
+    suffix = "_sonar"
+    parent_link="${namespace}/base_link"
+    topic = "${namespace}/sonar"
+    mass="0.02"
+    update_rate="15"
+    samples="100"
+    fov="1.54719755"
+    width = "120"
+    height ="120">
+    <inertia ixx="0.00001" ixy="0.0" ixz="0.0" iyy="0.00001" iyz="0.0" izz="0.00001" />
+    <origin xyz="1.15 0 0.4" rpy="0 0.6 0"/>
+  </xacro:forward_looking_sonar>
 </robot>

Commit message: added sidescan

File: rexrov2_description/urdf/rexrov2_sensors.xacro (robot description, xacro)
@@ -85,3 +85,7 @@
     <origin xyz="1.15 0 0.4" rpy="0 0.6 0"/>
   </xacro:forward_looking_sonar>
+  <xacro:sidescan_sonar
+      namespace="${namespace}" parent_link="${namespace}/base_link" suffix="sonar">
+      <origin xyz="1.15 0 0.4" rpy="0 0.6 0" />
+  </xacro:sidescan_sonar>
 </robot>

Commit message: sidescan sonar facing forward

File: rexrov2_description/urdf/rexrov2_sensors.xacro (robot description, xacro)
@@ -87,5 +87,5 @@
   <xacro:sidescan_sonar
       namespace="${namespace}" parent_link="${namespace}/base_link" suffix="sonar">
-      <origin xyz="1.15 0 0.4" rpy="0 0.6 0" />
+      <origin xyz="1.15 0 0.4" rpy="0 0 0" />
   </xacro:sidescan_sonar>
 </robot>
